File: hardware/kicad/Minty-sniffle/Minty-sniffle.kicad_sch (KiCad schematic)
At the start: 0 parts

Commit message: making a backup before shifting to altium
Parts:
- added BT1: BH1000G, BH1000G:BAT_BH1000G, symbol CR2477 holder:BH1000G
- added C1, C2, C3, C4, C5, C6, C7: ${VALUE}, symbol Capacitors:Capacitor - non polarized
- added D1: LED, symbol Device:LED
- added D2: BAT54A, Package_TO_SOT_SMD:SOT-23, symbol Diode:BAT54A
- added R1, R2, R3, R4, R5, R6, R7: ${VALUE}, symbol Resistors:Resistor
- added SW1: SW_Push, symbol Switch:SW_Push
- added U1: holyiot-18010, 18039:PCBComponent_1, symbol kleeb-master:holyiot-18010
- added U2: BME680, Package_LGA:Bosch_LGA-8_3x3mm_P0.8mm_ClockwisePinNumbering, symbol Sensor:BME680
- added U3: FM24CL16B-GTR, infineon fram ic:SOIC-8, symbol 2026-09-20_13-56-15:FM24CL16B-GTR
- added U4: (no value), Package_SO:SOIC-8_5.3x5.3mm_P1.27mm, symbol sd3031:SD3031
Connections:
- new net: U4.1 (f32k), U4.4 (4_nc)
- new net GND: U1.1 (GND), U1.32 (GND), U1.44 (GND)
Other:
- company: (none) -> Shourya Pandey
- title: (none) -> Minty-sniffle

Commit message: i am done for the day will do the connections of the some other day
Parts:
- removed U1: holyiot-18010, 18039:PCBComponent_1, symbol kleeb-master:holyiot-18010
- added U1: (no value), 18039:PCBComponent_1, symbol holyiot 18039:holyiot_18039
Connections:
- net GND: now also U1.78 (GND_3), U1.79 (GND_2), U1.94 (GND)

Commit message: finally the projects pcb is ready
Parts:
- removed C1, C2, C3, C4, C5, C6, C7: ${VALUE}, symbol Capacitors:Capacitor - non polarized
- removed D2: BAT54A, Package_TO_SOT_SMD:SOT-23, symbol Diode:BAT54A
- removed U1: (no value), 18039:PCBComponent_1, symbol holyiot 18039:holyiot_18039
- added 1: ISC-nRF52840-A, ISC-nRF52840-A-MODULE:ISC-nRF52840-MODULE, symbol ISC-nRF52840-A-MODULE:ISC-nRF52840-A-MODULE
- added C1: 220uF, MyLib:Capacitor_SMD__C_1206_3216Metric_Pad1.33x1.80mm_HandSolder_8506848e9f, symbol MySymbols:Device__C_Small_f867c60b3d
- added C2: 4.7uF, MyLib:Capacitor_SMD__C_1206_3216Metric_Pad1.33x1.80mm_HandSolder_8506848e9f, symbol MySymbols:Device__C_Small_f867c60b3d
- added C3, C4, C5, C6, C7, C9: 100nF, MyLib:Capacitor_SMD__C_1206_3216Metric_Pad1.33x1.80mm_HandSolder_8506848e9f, symbol MySymbols:Device__C_Small_f867c60b3d
- added C8: 10nF, MyLib:Capacitor_SMD__C_1206_3216Metric_Pad1.33x1.80mm_HandSolder_8506848e9f, symbol MySymbols:Device__C_Small_f867c60b3d
- added D3, D4, D5: BAT54J, MyLib:Diode_SMD__D_SOD-323_14c7701009, symbol MySymbols:Diode__BAT54J_f6754f6ea1
- added H1, H2, H3, H4: MountingHole, MyLib:MountingHole__MountingHole_2.2mm_M2_f6c03cebac, symbol MySymbols:Mechanical__MountingHole_7b31ad2790
- added J1: TC2030, MyLib:Connector__Tag-Connect_TC2030-IDC-NL_2x03_P1.27mm_Vertical_f22d01531a, symbol MySymbols:Connector_Generic__Conn_02x03_Odd_Even_bec5bf4a7c
- added Q1: AO3401A, MyLib:Package_TO_SOT_SMD__SOT-23_e3fc7a82cd, symbol MySymbols:Transistor_FET__AO3401A_2b0e6e3d18
- added Q2: 2N7002, MyLib:Package_TO_SOT_SMD__SOT-23_e3fc7a82cd, symbol MySymbols:Transistor_FET__2N7002_5844bcc8ad
- added R10, R11: 100k, MyLib:Resistor_SMD__R_1206_3216Metric_Pad1.30x1.75mm_HandSolder_5a326c096f, symbol Resistors:Resistor
- added R8: 10k, MyLib:Resistor_SMD__R_1206_3216Metric_Pad1.30x1.75mm_HandSolder_5a326c096f, symbol Resistors:Resistor
- added R9: 1k, MyLib:Resistor_SMD__R_1206_3216Metric_Pad1.30x1.75mm_HandSolder_5a326c096f, symbol Resistors:Resistor
- added SW2, SW3: SW_Push, ul_B31000p:B3U-1000P, symbol MySymbols:Switch__SW_Push_c280e58ffe
- added TP1: SYS_VBAT, MyLib:TestPoint__TestPoint_Pad_D1.0mm_9a299b34f1, symbol MySymbols:Connector__TestPoint_dec32a5d7d
- added TP2: GND, MyLib:TestPoint__TestPoint_Pad_D1.0mm_9a299b34f1, symbol MySymbols:Connector__TestPoint_dec32a5d7d
- added TP3: SDA, MyLib:TestPoint__TestPoint_Pad_D1.0mm_9a299b34f1, symbol MySymbols:Connector__TestPoint_dec32a5d7d
- added TP4: SCL, MyLib:TestPoint__TestPoint_Pad_D1.0mm_9a299b34f1, symbol MySymbols:Connector__TestPoint_dec32a5d7d
- added TP5: SWDIO, MyLib:TestPoint__TestPoint_Pad_D1.0mm_9a299b34f1, symbol MySymbols:Connector__TestPoint_dec32a5d7d
- added TP6: SWCLK, MyLib:TestPoint__TestPoint_Pad_D1.0mm_9a299b34f1, symbol MySymbols:Connector__TestPoint_dec32a5d7d
- added TP7: RESET, MyLib:TestPoint__TestPoint_Pad_D1.0mm_9a299b34f1, symbol MySymbols:Connector__TestPoint_dec32a5d7d
- D1: footprint (none) -> MyLib:LED_SMD__LED_1206_3216Metric_Pad1.42x1.75mm_HandSolder_5459fa1901; symbol Device:LED -> MySymbols:Device__LED_2376034a0a
- R1, R2: value ${VALUE} -> 4.7k; footprint (none) -> MyLib:Resistor_SMD__R_1206_3216Metric_Pad1.30x1.75mm_HandSolder_5a326c096f
- R3: value ${VALUE} -> 1k; footprint (none) -> MyLib:Resistor_SMD__R_1206_3216Metric_Pad1.30x1.75mm_HandSolder_5a326c096f
- R4: value ${VALUE} -> 2.2M; footprint (none) -> MyLib:Resistor_SMD__R_1206_3216Metric_Pad1.30x1.75mm_HandSolder_5a326c096f
- R5: value ${VALUE} -> 1M; footprint (none) -> MyLib:Resistor_SMD__R_1206_3216Metric_Pad1.30x1.75mm_HandSolder_5a326c096f
- R6, R7: value ${VALUE} -> 100k; footprint (none) -> MyLib:Resistor_SMD__R_1206_3216Metric_Pad1.30x1.75mm_HandSolder_5a326c096f
- SW1: footprint (none) -> ul_B31000p:B3U-1000P; symbol Switch:SW_Push -> MySymbols:Switch__SW_Push_c280e58ffe
- U2: footprint Package_LGA:Bosch_LGA-8_3x3mm_P0.8mm_ClockwisePinNumbering -> MyLib:Package_LGA__Bosch_LGA-8_3x3mm_P0.8mm_ClockwisePinNumbering_3a75655f61; symbol Sensor:BME680 -> MySymbols:Sensor__BME680_5fcc687010
- U4: footprint Package_SO:SOIC-8_5.3x5.3mm_P1.27mm -> MyLib:Package_SO__SOIC-8_5.3x5.3mm_P1.27mm_29768ff8c2
Connections:
- net GND: now also BT1.N, D1.1 (K), R5.2, R7.2, SW1.2, U2.1 (GND), U2.5 (SDO), U2.7 (GND), U3.4 (VSS), U3.7 (WP), U4.5 (Gnd), 1.1 (GND), 1.25 (GND), 1.37 (GND), C1.2, C2.2, C3.2, C4.2, C5.2, C6.2, C7.2, C8.2, J1.5 (Pin_5), Q2.2 (S), R11.2, SW3.2, TP2.1
- net SDA: now reaches U3.5 (SDA)
- net SDA: now also R1.2, U2.3 (SDI), U4.7 (Sda), 1.8 (P0.28), TP3.1
- net SCL: now reaches U3.6 (SCL)
- net SCL: now also R2.2, U2.4 (SCK), U4.8 (Scl), 1.9 (P0.29), TP4.1
- net SYS_VBAT: now reaches U3.8 (VDD)
- net SYS_VBAT: now also R1.1, R2.1, U2.2 (CSB), U2.6 (VDDIO), U2.8 (VDD), U4.2 (Vdd), 1.14 (VDD_NRF), C1.1, C2.1, C3.1, C4.1, C5.1, C6.1, C7.1, J1.1 (Pin_1), Q1.2 (S), R10.1, R11.1, R8.1, TP1.1
- net LED_A: now reaches D1.2 (A)
- net LED_A: now also R3.2
- net BUTTON: now reaches SW1.1
- net BUTTON: now also 1.17 (P0.12)
- net BAT+: now reaches R6.1
- net BAT+: now also BT1.P, R4.1, C9.1, Q1.3 (D)
- net PMOS_GATE: now reaches R6.2
- net PMOS_GATE: now also C9.2, D4.2 (A), Q1.1 (G), Q2.3 (D)
- net BAT_ADC: now reaches R4.2
- net BAT_ADC: now also R5.1, 1.7 (P0.02), C8.1
- net LED_GPIO: now reaches R3.1
- net LED_GPIO: now also 1.29 (P1.01)
- net NMOS_GATE: now reaches R7.1
- net NMOS_GATE: now also D3.1 (K), Q2.1 (G)
- new net: R8.2, SW2.1
- new net HOLD_DRIVE: D3.2 (A), R9.2
- new net PWR_BUTTON: 1.13 (P0.05), D5.2 (A), R10.2
- new net PWR_HOLD: 1.12 (P0.04), R9.1
- new net RESET: 1.21 (P0.18), J1.3 (Pin_3), SW2.2, TP7.1
- new net START_BUTTON: D4.1 (K), D5.1 (K), SW3.1
- new net SWCLK: 1.31 (SWDCLK), J1.4 (Pin_4), TP6.1
- new net SWDIO: 1.32 (SWDIO), J1.2 (Pin_2), TP5.1
- no-connect marks 0 -> 45
Other:
- note added: "BATTERY CONNECTOR"
- note added: "BATTERY DIVIDER"
- note added: "BUTTON: P0.05 reads active LOW through D5."
- note added: "DECOUPLING CAPACITOR"
- note added: "HOLD: P0.04 HIGH enables Q2 and Q1 after SW3 is released."
- note added: "Hold SW3 until firmware takes over; boot timing is firmware dependent."
- note added: "I2C PULLUPS"
- note added: "MCU"
- note added: "MCU SOFT POWER LATCH"
- note added: "MEMORY"
- note added: "Mounting"
- note added: "OFF current is nonzero; device leakage limits remain UNVERIFIED."
- note added: "OFF: save state; finish flash writes; disconnect BLE; drive P0.04 LOW."
- note added: "R11 discharges the rail and limits preserved BAT_ADC backfeed."
- note added: "RTC"
- note added: "Release SW3 for OFF. C9 gate-to-source keeps battery insertion OFF."
- note added: "SENSOR"
- note added: "START: press SW3; assert P0.04 HIGH early in boot."
- note added: "STATUS LED"
- note added: "SWD / RESET"
- note added: "TESTING POINTS"
- moved on the sheet: BT1, D1, R1, R2, R3, SW1, U2, U3, U4
